File: electronics/leg_thing/180513v1/leg_thing.sch (KiCad schematic (older format))
At the start: 8 parts, among them J1 HIP, J2 THIGH, J3 KNEE, J4 CALF, U1 ESP32THINGPOWERSHIELD, U2 Teensy3.2_no_outer_inner

Commit message: electronics: switching to 6 pin molex connectors
Parts:
- removed J1: HIP, Connectors_Terminal_Blocks:TerminalBlock_bornier-3_P5.08mm, symbol Screw_Terminal_01x03
- removed J2: THIGH, Connectors_Terminal_Blocks:TerminalBlock_bornier-3_P5.08mm, symbol Screw_Terminal_01x03
- removed J3: KNEE, Connectors_Terminal_Blocks:TerminalBlock_bornier-3_P5.08mm, symbol Screw_Terminal_01x03
- removed J4: CALF, Connectors_Terminal_Blocks:TerminalBlock_bornier-3_P5.08mm, symbol Screw_Terminal_01x03
- added J1: HIPCALF, leg_thing:MOLEX6PIN, symbol Conn_01x06_Male
- added J2: THIGHKNEE, leg_thing:MOLEX6PIN, symbol Conn_01x06_Male
- R1: value R -> 560; footprint Resistors_SMD:R_1206_HandSoldering -> Resistors_THT:R_Axial_DIN0207_L6.3mm_D2.5mm_P10.16mm_Horizontal
- R2: value R -> 1K; footprint Resistors_SMD:R_1206_HandSoldering -> Resistors_THT:R_Axial_DIN0207_L6.3mm_D2.5mm_P10.16mm_Horizontal
Connections:
- net +3V3: now also J1.3 (Pin_3), J2.1 (Pin_1), J2.5 (Pin_5)
- net +5V: now also J1.5 (Pin_5)
- net CALFPOT5V: now also J1.4 (Pin_4)
- net GND: now also J1.6 (Pin_6)
- net GNDA: now also J1.1 (Pin_1), J2.2 (Pin_2), J2.6 (Pin_6)
- net HIPPOT: now also J1.2 (Pin_2)
- net KNEEPOT: now also J2.4 (Pin_4)
- net THIGHPOT: now also J2.3 (Pin_3)
Changed lines of the file:
@@
 LIBS:leg_thing
 LIBS:teensy
+LIBS:leg_thing-cache
 EELAYER 25 0
 EELAYER END
@@
 P 9700 5350
 F 0 "R1" V 9780 5350 50  0000 C CNN
-F 1 "R" V 9700 5350 50  0000 C CNN
-F 2 "Resistors_SMD:R_1206_HandSoldering" V 9630 5350 50  0001 C CNN
+F 1 "560" V 9700 5350 50  0000 C CNN
+F 2 "Resistors_THT:R_Axial_DIN0207_L6.3mm_D2.5mm_P10.16mm_Horizontal" V 9630 5350 50  0001 C CNN
 F 3 "" H 9700 5350 50  0001 C CNN
 	1    9700 5350
@@
 P 9700 5650
 F 0 "R2" V 9780 5650 50  0000 C CNN
-F 1 "R" V 9700 5650 50  0000 C CNN
-F 2 "Resistors_SMD:R_1206_HandSoldering" V 9630 5650 50  0001 C CNN
+F 1 "1K" V 9700 5650 50  0000 C CNN
+F 2 "Resistors_THT:R_Axial_DIN0207_L6.3mm_D2.5mm_P10.16mm_Horizontal" V 9630 5650 50  0001 C CNN
 F 3 "" H 9700 5650 50  0001 C CNN
 	1    9700 5650
@@
 CALFPOT5V
 $Comp
-L Screw_Terminal_01x03 J1
-U 1 1 5AFA4AAE
-P 3150 4450
-F 0 "J1" H 3150 4650 50  0000 C CNN
-F 1 "HIP" H 3150 4250 50  0000 C CNN
-F 2 "Connectors_Terminal_Blocks:TerminalBlock_bornier-3_P5.08mm" H 3150 4450 50  0001 C CNN
-F 3 "" H 3150 4450 50  0001 C CNN
-	1    3150 4450
-	1    0    0    -1
-$EndComp
-$Comp
-L +3.3V #PWR010
-U 1 1 5AFA4B8E
-P 2800 4350
-F 0 "#PWR010" H 2800 4200 50  0001 C CNN
-F 1 "+3.3V" H 2800 4490 50  0000 C CNN
-F 2 "" H 2800 4350 50  0001 C CNN
-F 3 "" H 2800 4350 50  0001 C CNN
-	1    2800 4350
-	1    0    0    -1
-$EndComp
-$Comp
-L GNDA #PWR011
-U 1 1 5AFA4C9D
-P 2800 4550
-F 0 "#PWR011" H 2800 4300 50  0001 C CNN
-F 1 "GNDA" H 2800 4400 50  0000 C CNN
-F 2 "" H 2800 4550 50  0001 C CNN
-F 3 "" H 2800 4550 50  0001 C CNN
-	1    2800 4550
-	1    0    0    -1
-$EndComp
-Wire Wire Line
-	2800 4350 2950 4350
-Wire Wire Line
-	2800 4550 2950 4550
-Wire Wire Line
-	2950 4450 2550 4450
-Text Label 2550 4450 0    60   ~ 0
-HIPPOT
-$Comp
-L Screw_Terminal_01x03 J2
-U 1 1 5AFA4F24
-P 3150 5100
-F 0 "J2" H 3150 5300 50  0000 C CNN
-F 1 "THIGH" H 3150 4900 50  0000 C CNN
-F 2 "Connectors_Terminal_Blocks:TerminalBlock_bornier-3_P5.08mm" H 3150 5100 50  0001 C CNN
-F 3 "" H 3150 5100 50  0001 C CNN
-	1    3150 5100
-	1    0    0    -1
-$EndComp
-$Comp
-L +3.3V #PWR012
-U 1 1 5AFA4F2A
-P 2800 5000
-F 0 "#PWR012" H 2800 4850 50  0001 C CNN
-F 1 "+3.3V" H 2800 5140 50  0000 C CNN
-F 2 "" H 2800 5000 50  0001 C CNN
-F 3 "" H 2800 5000 50  0001 C CNN
-	1    2800 5000
-	1    0    0    -1
-$EndComp
-$Comp
-L GNDA #PWR013
-U 1 1 5AFA4F30
-P 2800 5200
-F 0 "#PWR013" H 2800 4950 50  0001 C CNN
-F 1 "GNDA" H 2800 5050 50  0000 C CNN
-F 2 "" H 2800 5200 50  0001 C CNN
-F 3 "" H 2800 5200 50  0001 C CNN
-	1    2800 5200
-	1    0    0    -1
-$EndComp
-Wire Wire Line
-	2800 5000 2950 5000
-Wire Wire Line
-	2800 5200 2950 5200
-Wire Wire Line
-	2950 5100 2550 5100
-Text Label 2550 5100 0    60   ~ 0
-THIGHPOT
-$Comp
-L Screw_Terminal_01x03 J3
-U 1 1 5AFA4F70
-P 3150 5750
-F 0 "J3" H 3150 5950 50  0000 C CNN
-F 1 "KNEE" H 3150 5550 50  0000 C CNN
-F 2 "Connectors_Terminal_Blocks:TerminalBlock_bornier-3_P5.08mm" H 3150 5750 50  0001 C CNN
-F 3 "" H 3150 5750 50  0001 C CNN
-	1    3150 5750
-	1    0    0    -1
-$EndComp
-$Comp
-L +3.3V #PWR014
-U 1 1 5AFA4F76
-P 2800 5650
-F 0 "#PWR014" H 2800 5500 50  0001 C CNN
-F 1 "+3.3V" H 2800 5790 50  0000 C CNN
-F 2 "" H 2800 5650 50  0001 C CNN
-F 3 "" H 2800 5650 50  0001 C CNN
-	1    2800 5650
-	1    0    0    -1
-$EndComp
-$Comp
-L GNDA #PWR015
-U 1 1 5AFA4F7C
-P 2800 5850
-F 0 "#PWR015" H 2800 5600 50  0001 C CNN
-F 1 "GNDA" H 2800 5700 50  0000 C CNN
-F 2 "" H 2800 5850 50  0001 C CNN
-F 3 "" H 2800 5850 50  0001 C CNN
-	1    2800 5850
-	1    0    0    -1
-$EndComp
-Wire Wire Line
-	2800 5650 2950 5650
-Wire Wire Line
-	2800 5850 2950 5850
-Wire Wire Line
-	2950 5750 2550 5750
-Text Label 2550 5750 0    60   ~ 0
-KNEEPOT
-$Comp
-L Screw_Terminal_01x03 J4
-U 1 1 5AFA4FAB
-P 3150 6400
-F 0 "J4" H 3150 6600 50  0000 C CNN
-F 1 "CALF" H 3150 6200 50  0000 C CNN
-F 2 "Connectors_Terminal_Blocks:TerminalBlock_bornier-3_P5.08mm" H 3150 6400 50  0001 C CNN
-F 3 "" H 3150 6400 50  0001 C CNN
-	1    3150 6400
-	1    0    0    -1
-$EndComp
-Wire Wire Line
-	2800 6300 2950 6300
-Wire Wire Line
-	2800 6500 2950 6500
-Wire Wire Line
-	2500 6400 2950 6400
-Text Label 2500 6400 0    60   ~ 0
-CALFPOT5V
-$Comp
-L GND #PWR016
+L GND #PWR010
 U 1 1 5AFA532B
 P 9700 5800
-F 0 "#PWR016" H 9700 5550 50  0001 C CNN
+F 0 "#PWR010" H 9700 5550 50  0001 C CNN
 F 1 "GND" H 9700 5650 50  0000 C CNN
 F 2 "" H 9700 5800 50  0001 C CNN
@@
 $EndComp
 $Comp
-L GND #PWR017
-U 1 1 5AFA5426
-P 2800 6500
-F 0 "#PWR017" H 2800 6250 50  0001 C CNN
-F 1 "GND" H 2800 6350 50  0000 C CNN
-F 2 "" H 2800 6500 50  0001 C CNN
-F 3 "" H 2800 6500 50  0001 C CNN
-	1    2800 6500
-	1    0    0    -1
-$EndComp
-$Comp
-L +5V #PWR018
-U 1 1 5AFA5531
-P 2800 6300
-F 0 "#PWR018" H 2800 6150 50  0001 C CNN
-F 1 "+5V" H 2800 6440 50  0000 C CNN
-F 2 "" H 2800 6300 50  0001 C CNN
-F 3 "" H 2800 6300 50  0001 C CNN
-	1    2800 6300
-	1    0    0    -1
-$EndComp
+L Conn_01x06_Male J1
+U 1 1 5B04B5B9
+P 4300 4600
+F 0 "J1" H 4300 4900 50  0000 C CNN
+F 1 "HIPCALF" H 4300 4200 50  0000 C CNN
+F 2 "leg_thing:MOLEX6PIN" H 4300 4600 50  0001 C CNN
+F 3 "" H 4300 4600 50  0001 C CNN
+	1    4300 4600
+	1    0    0    -1
+$EndComp
+$Comp
+L Conn_01x06_Male J2
+U 1 1 5B04B624
+P 4300 5600
+F 0 "J2" H 4300 5900 50  0000 C CNN
+F 1 "THIGHKNEE" H 4300 5200 50  0000 C CNN
+F 2 "leg_thing:MOLEX6PIN" H 4300 5600 50  0001 C CNN
+F 3 "" H 4300 5600 50  0001 C CNN
+	1    4300 5600
+	1    0    0    -1
+$EndComp
+Wire Wire Line
+	4500 4400 5600 4400
+Wire Wire Line
+	4500 4500 4700 4500
+Wire Wire Line
+	4500 4600 5300 4600
+Wire Wire Line
+	4500 4700 4700 4700
+Wire Wire Line
+	4500 4800 5300 4800
+Wire Wire Line
+	4500 4900 5300 4900
+Wire Wire Line
+	4500 5400 5450 5400
+Wire Wire Line
+	4500 5500 5450 5500
+Wire Wire Line
+	4500 5600 4700 5600
+Wire Wire Line
+	4500 5700 4700 5700
+Wire Wire Line
+	4500 5800 5200 5800
+Wire Wire Line
+	4500 5900 5200 5900
+Text Label 4700 4500 0    60   ~ 0
+HIPPOT
+Text Label 4700 4700 0    60   ~ 0
+CALFPOT5V
+$Comp
+L +5V #PWR011
+U 1 1 5B04BB18
+P 5300 4800
+F 0 "#PWR011" H 5300 4650 50  0001 C CNN
+F 1 "+5V" H 5300 4940 50  0000 C CNN
+F 2 "" H 5300 4800 50  0001 C CNN
+F 3 "" H 5300 4800 50  0001 C CNN
+	1    5300 4800
+	1    0    0    -1
+$EndComp
+$Comp
+L +3.3V #PWR012
+U 1 1 5B04BB4B
+P 5300 4600
+F 0 "#PWR012" H 5300 4450 50  0001 C CNN
+F 1 "+3.3V" H 5300 4740 50  0000 C CNN
+F 2 "" H 5300 4600 50  0001 C CNN
+F 3 "" H 5300 4600 50  0001 C CNN
+	1    5300 4600
+	1    0    0    -1
+$EndComp
+$Comp
+L GNDA #PWR013
+U 1 1 5B04BB74
+P 5600 4400
+F 0 "#PWR013" H 5600 4150 50  0001 C CNN
+F 1 "GNDA" H 5600 4250 50  0000 C CNN
+F 2 "" H 5600 4400 50  0001 C CNN
+F 3 "" H 5600 4400 50  0001 C CNN
+	1    5600 4400
+	1    0    0    -1
+$EndComp
+$Comp
+L GND #PWR014
+U 1 1 5B04BBBB
+P 5300 4900
+F 0 "#PWR014" H 5300 4650 50  0001 C CNN
+F 1 "GND" H 5300 4750 50  0000 C CNN
+F 2 "" H 5300 4900 50  0001 C CNN
+F 3 "" H 5300 4900 50  0001 C CNN
+	1    5300 4900
+	1    0    0    -1
+$EndComp
+Text Label 4700 5600 0    60   ~ 0
+THIGHPOT
+Text Label 4700 5700 0    60   ~ 0
+KNEEPOT
+$Comp
+L +3.3V #PWR015
+U 1 1 5B04BDC2
+P 5200 5800
+F 0 "#PWR015" H 5200 5650 50  0001 C CNN
+F 1 "+3.3V" H 5200 5940 50  0000 C CNN
+F 2 "" H 5200 5800 50  0001 C CNN
+F 3 "" H 5200 5800 50  0001 C CNN
+	1    5200 5800
+	1    0    0    -1
+$EndComp
+$Comp
+L GNDA #PWR016
+U 1 1 5B04BDEB
+P 5200 5900
+F 0 "#PWR016" H 5200 5650 50  0001 C CNN
+F 1 "GNDA" H 5200 5750 50  0000 C CNN
+F 2 "" H 5200 5900 50  0001 C CNN
+F 3 "" H 5200 5900 50  0001 C CNN
+	1    5200 5900
+	1    0    0    -1
+$EndComp
+$Comp
+L GNDA #PWR017
+U 1 1 5B04BE14
+P 5450 5500
+F 0 "#PWR017" H 5450 5250 50  0001 C CNN
+F 1 "GNDA" H 5450 5350 50  0000 C CNN
+F 2 "" H 5450 5500 50  0001 C CNN
+F 3 "" H 5450 5500 50  0001 C CNN
+	1    5450 5500
+	1    0    0    -1
+$EndComp
+$Comp
+L +3.3V #PWR018
+U 1 1 5B04BE47
+P 5450 5400
+F 0 "#PWR018" H 5450 5250 50  0001 C CNN
+F 1 "+3.3V" H 5450 5540 50  0000 C CNN
+F 2 "" H 5450 5400 50  0001 C CNN
+F 3 "" H 5450 5400 50  0001 C CNN
+	1    5450 5400
+	1    0    0    -1
+$EndComp

Commit message: adding pull-up resistor on disable line
Parts:
- added J3: SPI, Pin_Headers:Pin_Header_Straight_1x03_Pitch2.54mm, symbol Conn_01x03_Male
- added R3: 1K, Resistors_SMD:R_1206_HandSoldering, symbol R
Connections:
- net +3V3: now also R3.1
- net GND: now also J3.1 (Pin_1)
- net MDISABLE: now also R3.2
- net SPI_DO: now reaches U2.13 (11_DOUT)
- net SPI_DO: now also J3.3 (Pin_3)
- net SPI_CLK: now reaches U2.21 (14_A0_SCK)
- net SPI_CLK: now also J3.2 (Pin_2)
Changed lines of the file:
@@
 	3800 3050 4050 3050
 Wire Wire Line
-	3800 2350 3900 2350
+	3800 2350 4800 2350
 Wire Wire Line
 	3800 2250 3900 2250
@@
 Text Label 3900 2250 0    60   ~ 0
 HIP1
-Text Label 3900 2350 0    60   ~ 0
+Text Label 4800 2350 0    60   ~ 0
 MDISABLE
 $Comp
@@
 	1    0    0    -1
 $EndComp
+$Comp
+L Conn_01x03_Male J3
+U 1 1 5B09DE9E
+P 2600 4550
+F 0 "J3" H 2600 4750 50  0000 C CNN
+F 1 "SPI" H 2600 4350 50  0000 C CNN
+F 2 "Pin_Headers:Pin_Header_Straight_1x03_Pitch2.54mm" H 2600 4550 50  0001 C CNN
+F 3 "" H 2600 4550 50  0001 C CNN
+	1    2600 4550
+	1    0    0    -1
+$EndComp
+Wire Wire Line
+	2800 4450 3550 4450
+Wire Wire Line
+	2800 4550 3050 4550
+Wire Wire Line
+	2800 4650 3050 4650
+Text Label 3050 4650 0    60   ~ 0
+SPI_DO
+Text Label 3050 4550 0    60   ~ 0
+SPI_CLK
+$Comp
+L GND #PWR019
+U 1 1 5B09E09B
+P 3550 4450
+F 0 "#PWR019" H 3550 4200 50  0001 C CNN
+F 1 "GND" H 3550 4300 50  0000 C CNN
+F 2 "" H 3550 4450 50  0001 C CNN
+F 3 "" H 3550 4450 50  0001 C CNN
+	1    3550 4450
+	1    0    0    -1
+$EndComp
+Wire Wire Line
+	6800 2850 6250 2850
+Text Label 6250 2850 0    60   ~ 0
+SPI_DO
+Wire Wire Line
+	6800 3650 6250 3650
+Text Label 6250 3650 0    60   ~ 0
+SPI_CLK
+$Comp
+L R R3
+U 1 1 5B0AA829
+P 4500 2200
+F 0 "R3" V 4580 2200 50  0000 C CNN
+F 1 "1K" V 4500 2200 50  0000 C CNN
+F 2 "Resistors_SMD:R_1206_HandSoldering" V 4430 2200 50  0001 C CNN
+F 3 "" H 4500 2200 50  0001 C CNN
+	1    4500 2200
+	1    0    0    -1
+$EndComp
+$Comp
+L +3.3V #PWR020
+U 1 1 5B0AA9A7
+P 4500 2050
+F 0 "#PWR020" H 4500 1900 50  0001 C CNN
+F 1 "+3.3V" H 4500 2190 50  0000 C CNN
+F 2 "" H 4500 2050 50  0001 C CNN
+F 3 "" H 4500 2050 50  0001 C CNN
+	1    4500 2050
+	1    0    0    -1
+$EndComp
+Connection ~ 4500 2350
 $EndSCHEMATC
