Commit message: calf load and imu (needs verification) working in sim

File: stompy/simulation/data/stompy.urdf (robot description, URDF)
Before this commit: robot stompy, 37 links, 36 joints
Joints:
- joint stompy__fl_leg__calf_upper_to_calf_lower: limit lower=-0.104 upper=0 effort=0 velocity=0.0 -> lower=0.0 upper=0.104 effort=5337 velocity=0.0
- joint stompy__fr_leg__calf_upper_to_calf_lower: limit lower=-0.104 upper=0.104 effort=10942 velocity=0.0 -> lower=0.0 upper=0.104 effort=5337 velocity=0.0
- joint stompy__ml_leg__calf_upper_to_calf_lower: limit lower=-0.104 upper=0.104 effort=10942 velocity=0.0 -> lower=0.0 upper=0.104 effort=5337 velocity=0.0
- joint stompy__mr_leg__calf_upper_to_calf_lower: limit lower=-0.104 upper=0.104 effort=10942 velocity=0.0 -> lower=0.0 upper=0.104 effort=5337 velocity=0.0
- joint stompy__rl_leg__calf_upper_to_calf_lower: limit lower=-0.104 upper=0.104 effort=10942 velocity=0.0 -> lower=0.0 upper=0.104 effort=5337 velocity=0.0
- joint stompy__rr_leg__calf_upper_to_calf_lower: limit lower=-0.104 upper=0.104 effort=10942 velocity=0.0 -> lower=0.0 upper=0.104 effort=5337 velocity=0.0
